File: RevA.sch (KiCad schematic (older format))
At the start: 30 parts, among them P1 ELECTODES, U1 LM358, X1 16MHz

Commit message: Updated Schems
Parts:
- removed C? (x4): C, ~, symbol C
- removed Q?: MOSFET_N, ~, symbol MOSFET_N
- removed U?: DS1337C, symbol DS1337C
- added BT1, BT2: BATTERY, ~, symbol BATTERY
- added C10, C7, C8, C9: 10uF, ~, symbol CP
- added D1, D2: DIODE, ~, symbol DIODE
- added D3: LED, ~, symbol LED
- added R1, R10, R11, R12: 10k, ~, symbol R
- added R13: 150, ~, symbol R
- added SW1: Power Switch, ~, symbol SWITCH_INV
- added U6: PCF8563, symbol PCF8563
- added X2: 32.768kHz, ~, symbol CRYSTAL
- C3, C4, C5, C6: renamed from C?; value C -> .22uF
- P1: renamed from P?; value CONN_3X2 -> ICSP
- R2, R7: renamed from R?; value R -> 10k
- R3, R4: renamed from R?; value R -> 2.2k
- R5, R6: renamed from R?; value R -> 13k
- R8: renamed from R?; value R -> 10M
- R9: renamed from R?; value R -> 470
- RV1: renamed from RV?; value POT -> 20k
- gave numbers to parts that had none: 5
- renumbered P1 to P2
Connections:
- net labels added: INT, MISO, MOSI, RST, RTC_SCL, RTC_SDA, SCK, led
- net labels removed: potSCK, potSI
- wire segments 59 -> 100
Other:
- note added: "Current Regulator\n"
- note added: "Digital Potentiometer\n"
- note added: "MCU and Programming\n"
- note added: "Misc."
- note added: "Oscillator\n"
- note added: "Power\n"
- note added: "Real Time Clock"
- moved on the sheet: C1, C2, C6, IC1, P1, P2, R7, R8, R9, U2A, U3, U4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
